File: untitled.brd (EAGLE design)
At the start: 100 x 80 mm, 43 parts, among them IC1 MCP604SL, IC2 TL072D, U1 TEXAS_INSTRUMENTS_DAC8531E-25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, U2 L79L05ACUTRL79L05ACU, U4 MCP1501-40E/SN, U5 MC7805CDT, U6 MCP3204-CI-SL, X1 1751251, X2 PN61729-S

Commit message: dodano zlacze programatora i rezystor nastawny
Parts:
- removed H6: MOUNT-PAD-ROUND4.3, holes:4,3-PAD
- removed R13, R14: 10k, rcl:M1206
- added R15: (no value), rcl:RTRIM64Y
- added SV1: (no value), con-harting-ml:ML10
- moved X2 19.3 mm to (66.0, 19.1), turned to 0 degrees
- moved C6 3.81 mm to (49.5, 31.8)
- moved R1 2.84 mm to (66.0, 27.9)
- moved R2 2.84 mm to (66.0, 30.5)
- moved R7 1.55 mm to (45.5, 39.6)
- moved C8 1.27 mm to (58.4, 31.8), turned to 0 degrees
Connections:
- removed net ADC-DOUT: U$1.11, U6.10
- removed net DATA: U$1.10, U1.7, U6.9
- removed net N$12: R7.1, U$1.13
- new net MISO: SV1.9, U$1.11, U6.10
- new net MOSI: SV1.1, U$1.10, U1.7, U6.9
- new net RST: R7.1, SV1.5, U$1.13
- net CLK: now also SV1.7
- net GND: now also SV1.10, SV1.4, SV1.6, SV1.8; no longer H6.B4,3
- net N$22: now also R15.2; no longer R13.1, R14.2
- net N$6: now also R15.1; no longer R14.1
- net VREF: now also R15.3; no longer R13.2
Routing:
- net MISO: track 0.00 -> 85.7 mm, vias 0 -> 3
- net MOSI: track 0.00 -> 75.1 mm, vias 0 -> 2
- net RST: track 0.00 -> 58.2 mm, vias 0 -> 2
- net CLK: track 47.3 -> 97.6 mm, vias 2 -> 3
- net DATA: track 42.7 -> 0.00 mm
- net -15V: track 58.5 -> 77.3 mm
- net ADC-DOUT: track 18.7 -> 0.00 mm, vias 2 -> 0
- net N$8: track 43.2 -> 26.0 mm
- net N$12: track 9.76 -> 0.00 mm
- net VCC: track 222.0 -> 214.9 mm
- net N$3: track 13.6 -> 18.4 mm
- net N$4: track 29.1 -> 24.7 mm
- net GND: track 101.4 -> 104.6 mm
- net N$14: track 20.6 -> 17.8 mm
- net N$2: track 27.1 -> 24.4 mm
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- added copper zone on layer 1, net POL
- removed copper zone on layer 1, net POLYGON

Commit message: poprawki
Parts:
- added H6: MOUNT-PAD-ROUND4.3, holes:4,3-PAD
- moved X1 13.9 mm to (46.5, 4.57)
- moved C1 12.1 mm to (79.5, 41.4)
- moved C4 10.8 mm to (85.9, 50.3)
- moved SV1 10.7 mm to (85.9, 19.8), flipped to the bottom
- moved R15 9.56 mm to (70.6, 40.1)
- moved U2 9.56 mm to (83.3, 37.6)
- moved C5 9.56 mm to (38.9, 43.9)
- moved H1 9.56 mm to (25.4, 63.6)
- moved H3 9.56 mm to (10.9, 63.6)
- moved H4 9.56 mm to (40.1, 63.6)
- moved R7 9.56 mm to (43.7, 30.2)
- moved U4 9.56 mm to (52.8, 37.6)
- moved X2 9.56 mm to (64.3, 9.65)
- moved C7 9.56 mm to (31.8, 10.4)
- moved H2 9.56 mm to (74.7, 63.8)
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Connections:
- net GND: now also H6.B4,3
Routing:
- net VDD: track 37.7 -> 50.8 mm
- net GND: track 104.6 -> 96.6 mm
- net MOSI: track 75.1 -> 82.1 mm
- net RST: track 58.2 -> 62.5 mm
- net CLK: track 97.6 -> 101.8 mm
- net +15V: track 24.7 -> 22.2 mm
- net MISO: track 85.7 -> 87.5 mm
- net VCC: track 214.9 -> 213.2 mm
- removed copper zone on layer 1, net POL
Other:
- board size 100 x 80 mm -> 94.9 x 69.8 mm

Commit message: poprawki
Routing:
- net CLK: track 101.8 -> 103.0 mm
Changed lines of the file:
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@@
 <contactref element="H6" pad="B4,3"/>
 <wire x1="88.138" y1="63.754" x2="88.138" y2="56.134" width="0.4064" layer="1"/>
-<wire x1="30.582" y1="15.282" x2="36.982" y2="15.282" width="0" layer="19" extent="1-1"/>
 </signal>
 <signal name="N$1">
@@
 <contactref element="X1" pad="3"/>
 <contactref element="U5" pad="1"/>
-<wire x1="40.2245" y1="7.4295" x2="21.9755" y2="7.4295" width="0.6096" layer="1"/>
+<wire x1="36.4145" y1="7.4295" x2="21.9755" y2="7.4295" width="0.6096" layer="1"/>
 <wire x1="21.912" y1="7.366" x2="21.9755" y2="7.4295" width="0.4064" layer="1"/>
-<wire x1="42.982" y1="4.672" x2="40.2245" y2="7.4295" width="0.6096" layer="1"/>
+<wire x1="42.982" y1="4.672" x2="39.172" y2="4.672" width="0.6096" layer="1"/>
+<wire x1="39.172" y1="4.672" x2="36.4145" y2="7.4295" width="0.6096" layer="1"/>
 </signal>
 <signal name="-15V">
@@
 <contactref element="SV1" pad="7"/>
 <contactref element="U1" pad="6"/>
-<wire x1="45.212" y1="24.13" x2="45.212" y2="12.192" width="0.4064" layer="16"/>
-<via x="45.212" y="12.192" extent="1-16" drill="1.397"/>
-<wire x1="61.722" y1="9.652" x2="59.182" y2="12.192" width="0.4064" layer="1"/>
-<wire x1="61.722" y1="9.652" x2="66.802" y2="9.652" width="0.4064" layer="1"/>
-<wire x1="45.212" y1="12.192" x2="59.182" y2="12.192" width="0.4064" layer="1"/>
+<wire x1="45.212" y1="24.13" x2="45.212" y2="11.176" width="0.4064" layer="16"/>
+<via x="45.212" y="11.176" extent="1-16" drill="1.397"/>
+<wire x1="66.802" y1="9.652" x2="61.722" y2="9.652" width="0.4064" layer="1"/>
 <wire x1="66.802" y1="9.652" x2="75.692" y2="18.542" width="0.4064" layer="1"/>
 <wire x1="42.812" y1="23.482" x2="43.46" y2="24.13" width="0.4064" layer="1"/>
@@
 <wire x1="85.852" y1="18.542" x2="75.692" y2="18.542" width="0.4064" layer="1"/>
 <wire x1="85.852" y1="18.542" x2="87.122" y2="17.272" width="0.4064" layer="1"/>
+<wire x1="51.562" y1="11.938" x2="50.8" y2="11.176" width="0.4064" layer="1"/>
+<wire x1="50.8" y1="11.176" x2="45.212" y2="11.176" width="0.4064" layer="1"/>
+<wire x1="61.722" y1="9.652" x2="59.436" y2="11.938" width="0.4064" layer="1"/>
+<wire x1="59.436" y1="11.938" x2="51.562" y2="11.938" width="0.4064" layer="1"/>
 </signal>
 <signal name="N$11">
@@
 <wire x1="52.832" y1="31.242" x2="53.807" y2="32.217" width="0.4064" layer="1"/>
 <via x="52.832" y="31.242" extent="1-16" drill="1.397"/>
-<wire x1="52.832" y1="31.242" x2="52.832" y2="14.732" width="0.4064" layer="16"/>
-<via x="52.832" y="14.732" extent="1-16" drill="1.397"/>
-<wire x1="52.832" y1="14.732" x2="42.672" y2="14.732" width="0.4064" layer="1"/>
-<wire x1="42.672" y1="14.732" x2="40.132" y2="12.192" width="0.4064" layer="1"/>
+<wire x1="52.832" y1="31.242" x2="52.578" y2="30.988" width="0.4064" layer="16"/>
+<wire x1="52.578" y1="30.988" x2="52.578" y2="14.224" width="0.4064" layer="16"/>
+<via x="52.578" y="14.224" extent="1-16" drill="1.397"/>
+<wire x1="52.578" y1="14.224" x2="42.164" y2="14.224" width="0.4064" layer="1"/>
+<wire x1="42.164" y1="14.224" x2="40.132" y2="12.192" width="0.4064" layer="1"/>
 <wire x1="36.322" y1="12.192" x2="40.132" y2="12.192" width="0.4064" layer="1"/>
 <contactref element="U$1" pad="41"/>
@@
 <wire x1="41.91" y1="26.162" x2="41.656" y2="25.908" width="0.4064" layer="16"/>
 <contactref element="SV1" pad="9"/>
-<wire x1="41.656" y1="25.908" x2="41.656" y2="10.414" width="0.4064" layer="16"/>
-<via x="41.656" y="10.414" extent="1-16" drill="1.397"/>
-<wire x1="41.656" y1="10.414" x2="54.61" y2="10.414" width="0.4064" layer="1"/>
-<wire x1="54.61" y1="10.414" x2="55.372" y2="9.652" width="0.4064" layer="1"/>
-<wire x1="55.372" y1="9.652" x2="55.372" y2="7.112" width="0.4064" layer="1"/>
+<wire x1="41.656" y1="25.908" x2="41.656" y2="9.398" width="0.4064" layer="16"/>
+<via x="41.656" y="9.398" extent="1-16" drill="1.397"/>
+<wire x1="41.656" y1="9.398" x2="55.372" y2="9.398" width="0.4064" layer="1"/>
+<wire x1="55.372" y1="9.398" x2="55.372" y2="7.112" width="0.4064" layer="1"/>
 <wire x1="55.372" y1="7.112" x2="56.642" y2="5.842" width="0.4064" layer="1"/>
 <wire x1="56.642" y1="5.842" x2="76.962" y2="5.842" width="0.4064" layer="1"/>

Commit message: poprawki
Parts:
- added H10, H7, H8, H9: MOUNT-PAD-ROUND2.8, holes:2,8-PAD
- H1, H2, H3, H4, H5, H6: value MOUNT-PAD-ROUND4.3 -> MOUNT-PAD-ROUND2.8; device holes:4,3-PAD -> holes:2,8-PAD
- R15: device rcl:RTRIM64Y -> rcl-moja:RTRIM64Y
- moved H6 6.10 mm to (82.0, 63.8)
- moved H5 5.08 mm to (59.2, 63.5)
- moved H4 2.54 mm to (42.7, 63.6)
- moved H3 0.76 mm to (10.2, 63.6)
- moved U4 0.76 mm to (52.8, 38.4)
Connections:
- net ADC-IN0: now also H1.B2,8; no longer H1.B4,3
- net ADC-IN1: now also H3.B2,8; no longer H3.B4,3
- net ADC-IN2: now also H5.B2,8; no longer H5.B4,3
- net ADC-IN3: now also H4.B2,8; no longer H4.B4,3
- net GND: now also H10.B2,8, H6.B2,8, H7.B2,8, H8.B2,8, H9.B2,8; no longer H6.B4,3
- net N$6: now also H2.B2,8; no longer H2.B4,3
Routing:
- net GND: track 96.6 -> 87.7 mm
- net ADC-IN2: track 9.27 -> 13.6 mm
- net VREF: track 68.4 -> 72.2 mm
- net ADC-CH1: track 51.2 -> 53.2 mm
- net CLK: track 103.0 -> 104.8 mm
- net VDD: track 50.8 -> 52.1 mm
- net ADC-IN3: track 9.40 -> 10.6 mm
- net SYNC-DAC: track 42.4 -> 43.5 mm
- net N$19: track 65.9 -> 65.2 mm
- net VCC: track 213.2 -> 212.7 mm
Other:
- board text added: "PDG-2019"
- board text removed: "PG-2019"
