File: untitled.sch (EAGLE design)
At the start: 43 parts, among them IC1 MCP604SL, IC2 TL072D, U1 TEXAS_INSTRUMENTS_DAC8531E-25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, U2 L79L05ACUTRL79L05ACU, U4 MCP1501-40E/SN, U5 MC7805CDT, U6 MCP3204-CI-SL, X1 1751251, X2 PN61729-S

Commit message: dodano zlacze programatora i rezystor nastawny
Parts:
- removed H6: MOUNT-PAD-ROUND4.3, holes:MOUNT-PAD-ROUND4.3
- removed R13, R14: 10k, rcl:R-EU_M1206
- added R15: (no value), rcl:R-TRIMM64Y
- added SV1: (no value), con-harting-ml:ML10
Connections:
- removed net ADC-DOUT: U$1.PB3(PDO/MISO), U6.DOUT
- removed net DATA: U$1.PB2(PDI/MOSI), U1.DIN, U6.DIN
- removed net N$12: R7.1, U$1./RESET
- new net MISO: SV1.9, U$1.PB3(PDO/MISO), U6.DOUT
- new net MOSI: SV1.1, U$1.PB2(PDI/MOSI), U1.DIN, U6.DIN
- new net RST: R7.1, SV1.5, U$1./RESET
- net CLK: now also SV1.7
- net GND: now also SV1.10, SV1.4, SV1.6, SV1.8; no longer H6.MOUNT
- net N$22: now also R15.S; no longer R13.1, R14.2
- net N$6: now also R15.A; no longer R14.1
- net VREF: now also R15.E; no longer R13.2

Commit message: poprawki
Parts:
- added H6: MOUNT-PAD-ROUND4.3, holes:MOUNT-PAD-ROUND4.3
Connections:
- net GND: now also H6.MOUNT
Changed lines of the file:
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@@
 <part name="SV1" library="con-harting-ml" library_urn="urn:adsk.eagle:library:149" deviceset="ML10" device="" package3d_urn="urn:adsk.eagle:package:6967/1"/>
 <part name="SUPPLY13" library="supply2" library_urn="urn:adsk.eagle:library:372" deviceset="GND" device=""/>
+<part name="H6" library="holes" library_urn="urn:adsk.eagle:library:237" deviceset="MOUNT-PAD-ROUND" device="4.3" package3d_urn="urn:adsk.eagle:package:14286/1"/>
 </parts>
 <sheets>
@@
 <attribute name="VALUE" x="-1.905" y="-51.435" size="1.778" layer="96"/>
 </instance>
+<instance part="H6" gate="G$1" x="-60.96" y="134.62" smashed="yes" rot="R270">
+<attribute name="NAME" x="-60.3758" y="131.826" size="1.778" layer="95" rot="R270"/>
+</instance>
 </instances>
 <busses>
@@
 <pinref part="C4" gate="G$1" pin="-"/>
 <wire x1="-83.82" y1="144.78" x2="-76.2" y2="144.78" width="0.1524" layer="91"/>
-<wire x1="-76.2" y1="144.78" x2="-58.42" y2="144.78" width="0.1524" layer="91"/>
+<wire x1="-76.2" y1="144.78" x2="-60.96" y2="144.78" width="0.1524" layer="91"/>
+<wire x1="-60.96" y1="144.78" x2="-58.42" y2="144.78" width="0.1524" layer="91"/>
 <wire x1="-91.44" y1="144.78" x2="-91.44" y2="139.7" width="0.1524" layer="91"/>
 <junction x="-119.38" y="144.78"/>
@@
 <pinref part="U2" gate="G$0" pin="GND"/>
 <wire x1="-119.38" y1="144.78" x2="-119.38" y2="134.62" width="0.1524" layer="91"/>
+<pinref part="H6" gate="G$1" pin="MOUNT"/>
+<wire x1="-60.96" y1="137.16" x2="-60.96" y2="144.78" width="0.1524" layer="91"/>
+<junction x="-60.96" y="144.78"/>
 </segment>
 <segment>

Commit message: poprawki
Parts:
- added H10, H7, H8, H9: MOUNT-PAD-ROUND2.8, holes:MOUNT-PAD-ROUND2.8
- H1, H2, H3, H4, H5, H6: value MOUNT-PAD-ROUND4.3 -> MOUNT-PAD-ROUND2.8; device holes:MOUNT-PAD-ROUND4.3 -> holes:MOUNT-PAD-ROUND2.8
- R15: device rcl:R-TRIMM64Y -> rcl-moja:R-TRIMM64Y
Connections:
- net GND: now also H10.MOUNT, H7.MOUNT, H8.MOUNT, H9.MOUNT
Other:
- moved on the sheet: H6
Changed lines of the file:
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@@
 <part name="R5" library="rcl" library_urn="urn:adsk.eagle:library:334" deviceset="R-EU_" device="M1206" package3d_urn="urn:adsk.eagle:package:23566/1"/>
 <part name="R6" library="rcl" library_urn="urn:adsk.eagle:library:334" deviceset="R-EU_" device="M1206" package3d_urn="urn:adsk.eagle:package:23566/1"/>
-<part name="H1" library="holes" library_urn="urn:adsk.eagle:library:237" deviceset="MOUNT-PAD-ROUND" device="4.3" package3d_urn="urn:adsk.eagle:package:14286/1"/>
+<part name="H1" library="holes" library_urn="urn:adsk.eagle:library:237" deviceset="MOUNT-PAD-ROUND" device="2.8" package3d_urn="urn:adsk.eagle:package:14281/1" value="MOUNT-PAD-ROUND2.8"/>
 <part name="SUPPLY5" library="supply2" library_urn="urn:adsk.eagle:library:372" deviceset="GND" device=""/>
 <part name="P+4" library="supply1" library_urn="urn:adsk.eagle:library:371" deviceset="VCC" device=""/>
@@
 <attribute name="SPICEPREFIX" value="J"/>
 </part>
-<part name="H2" library="holes" library_urn="urn:adsk.eagle:library:237" deviceset="MOUNT-PAD-ROUND" device="4.3" package3d_urn="urn:adsk.eagle:package:14286/1"/>
+<part name="H2" library="holes" library_urn="urn:adsk.eagle:library:237" deviceset="MOUNT-PAD-ROUND" device="2.8" package3d_urn="urn:adsk.eagle:package:14281/1" value="MOUNT-PAD-ROUND2.8"/>
 <part name="P+6" library="supply1" library_urn="urn:adsk.eagle:library:371" deviceset="VCC" device=""/>
 <part name="C5" library="rcl" library_urn="urn:adsk.eagle:library:334" deviceset="C-EU" device="C0805K" package3d_urn="urn:adsk.eagle:package:23681/2" value="100n"/>
@@
 <part name="R4" library="rcl" library_urn="urn:adsk.eagle:library:334" deviceset="R-EU_" device="M1206" package3d_urn="urn:adsk.eagle:package:23566/1"/>
 <part name="R8" library="rcl" library_urn="urn:adsk.eagle:library:334" deviceset="R-EU_" device="M1206" package3d_urn="urn:adsk.eagle:package:23566/1"/>
-<part name="H3" library="holes" library_urn="urn:adsk.eagle:library:237" deviceset="MOUNT-PAD-ROUND" device="4.3" package3d_urn="urn:adsk.eagle:package:14286/1"/>
+<part name="H3" library="holes" library_urn="urn:adsk.eagle:library:237" deviceset="MOUNT-PAD-ROUND" device="2.8" package3d_urn="urn:adsk.eagle:package:14281/1" value="MOUNT-PAD-ROUND2.8"/>
 <part name="SUPPLY12" library="supply2" library_urn="urn:adsk.eagle:library:372" deviceset="GND" device=""/>
 <part name="D2" library="Vishay Semiconductor - MMSZ5231B-E3-08" deviceset="MMSZ5231B" device="VISHAY_SEMICONDUCTOR_MMSZ5231B-E3-08_0_0"/>
 <part name="R9" library="rcl" library_urn="urn:adsk.eagle:library:334" deviceset="R-EU_" device="M1206" package3d_urn="urn:adsk.eagle:package:23566/1"/>
 <part name="R10" library="rcl" library_urn="urn:adsk.eagle:library:334" deviceset="R-EU_" device="M1206" package3d_urn="urn:adsk.eagle:package:23566/1"/>
-<part name="H4" library="holes" library_urn="urn:adsk.eagle:library:237" deviceset="MOUNT-PAD-ROUND" device="4.3" package3d_urn="urn:adsk.eagle:package:14286/1"/>
+<part name="H4" library="holes" library_urn="urn:adsk.eagle:library:237" deviceset="MOUNT-PAD-ROUND" device="2.8" package3d_urn="urn:adsk.eagle:package:14281/1" value="MOUNT-PAD-ROUND2.8"/>
 <part name="SUPPLY14" library="supply2" library_urn="urn:adsk.eagle:library:372" deviceset="GND" device=""/>
 <part name="D3" library="Vishay Semiconductor - MMSZ5231B-E3-08" deviceset="MMSZ5231B" device="VISHAY_SEMICONDUCTOR_MMSZ5231B-E3-08_0_0"/>
 <part name="R11" library="rcl" library_urn="urn:adsk.eagle:library:334" deviceset="R-EU_" device="M1206" package3d_urn="urn:adsk.eagle:package:23566/1"/>
 <part name="R12" library="rcl" library_urn="urn:adsk.eagle:library:334" deviceset="R-EU_" device="M1206" package3d_urn="urn:adsk.eagle:package:23566/1"/>
-<part name="H5" library="holes" library_urn="urn:adsk.eagle:library:237" deviceset="MOUNT-PAD-ROUND" device="4.3" package3d_urn="urn:adsk.eagle:package:14286/1"/>
+<part name="H5" library="holes" library_urn="urn:adsk.eagle:library:237" deviceset="MOUNT-PAD-ROUND" device="2.8" package3d_urn="urn:adsk.eagle:package:14281/1" value="MOUNT-PAD-ROUND2.8"/>
 <part name="SUPPLY16" library="supply2" library_urn="urn:adsk.eagle:library:372" deviceset="GND" device=""/>
 <part name="D4" library="Vishay Semiconductor - MMSZ5231B-E3-08" deviceset="MMSZ5231B" device="VISHAY_SEMICONDUCTOR_MMSZ5231B-E3-08_0_0"/>
@@
 <part name="SUPPLY8" library="supply2" library_urn="urn:adsk.eagle:library:372" deviceset="VDD" device=""/>
 <part name="SUPPLY11" library="supply2" library_urn="urn:adsk.eagle:library:372" deviceset="VDD" device=""/>
-<part name="R15" library="rcl" library_urn="urn:adsk.eagle:library:334" deviceset="R-TRIMM" device="64Y" package3d_urn="urn:adsk.eagle:package:23750/1"/>
+<part name="R15" library="rcl-moja" deviceset="R-TRIMM" device="64Y" package3d_urn="urn:adsk.eagle:package:23750/1"/>
 <part name="SV1" library="con-harting-ml" library_urn="urn:adsk.eagle:library:149" deviceset="ML10" device="" package3d_urn="urn:adsk.eagle:package:6967/1"/>
 <part name="SUPPLY13" library="supply2" library_urn="urn:adsk.eagle:library:372" deviceset="GND" device=""/>
-<part name="H6" library="holes" library_urn="urn:adsk.eagle:library:237" deviceset="MOUNT-PAD-ROUND" device="4.3" package3d_urn="urn:adsk.eagle:package:14286/1"/>
+<part name="H6" library="holes" library_urn="urn:adsk.eagle:library:237" deviceset="MOUNT-PAD-ROUND" device="2.8" package3d_urn="urn:adsk.eagle:package:14281/1" value="MOUNT-PAD-ROUND2.8"/>
+<part name="H7" library="holes" library_urn="urn:adsk.eagle:library:237" deviceset="MOUNT-PAD-ROUND" device="2.8" package3d_urn="urn:adsk.eagle:package:14281/1" value="MOUNT-PAD-ROUND2.8"/>
+<part name="H8" library="holes" library_urn="urn:adsk.eagle:library:237" deviceset="MOUNT-PAD-ROUND" device="2.8" package3d_urn="urn:adsk.eagle:package:14281/1" value="MOUNT-PAD-ROUND2.8"/>
+<part name="H9" library="holes" library_urn="urn:adsk.eagle:library:237" deviceset="MOUNT-PAD-ROUND" device="2.8" package3d_urn="urn:adsk.eagle:package:14281/1" value="MOUNT-PAD-ROUND2.8"/>
+<part name="H10" library="holes" library_urn="urn:adsk.eagle:library:237" deviceset="MOUNT-PAD-ROUND" device="2.8" package3d_urn="urn:adsk.eagle:package:14281/1" value="MOUNT-PAD-ROUND2.8"/>
 </parts>
 <sheets>
@@
 <attribute name="VALUE" x="-1.905" y="-51.435" size="1.778" layer="96"/>
 </instance>
-<instance part="H6" gate="G$1" x="-60.96" y="134.62" smashed="yes" rot="R270">
-<attribute name="NAME" x="-60.3758" y="131.826" size="1.778" layer="95" rot="R270"/>
+<instance part="H6" gate="G$1" x="-66.04" y="139.7" smashed="yes" rot="R180">
+<attribute name="NAME" x="-68.834" y="139.1158" size="1.778" layer="95" rot="R180"/>
+</instance>
+<instance part="H7" gate="G$1" x="-66.04" y="132.08" smashed="yes" rot="R180">
+<attribute name="NAME" x="-68.834" y="131.4958" size="1.778" layer="95" rot="R180"/>
+</instance>
+<instance part="H8" gate="G$1" x="-55.88" y="139.7" smashed="yes">
+<attribute name="NAME" x="-53.086" y="140.2842" size="1.778" layer="95"/>
+</instance>
+<instance part="H9" gate="G$1" x="-55.88" y="132.08" smashed="yes">
+<attribute name="NAME" x="-53.086" y="132.6642" size="1.778" layer="95"/>
+</instance>
+<instance part="H10" gate="G$1" x="-60.96" y="152.4" smashed="yes" rot="R90">
+<attribute name="NAME" x="-61.5442" y="155.194" size="1.778" layer="95" rot="R90"/>
 </instance>
 </instances>
@@
 <wire x1="-119.38" y1="144.78" x2="-119.38" y2="134.62" width="0.1524" layer="91"/>
 <pinref part="H6" gate="G$1" pin="MOUNT"/>
-<wire x1="-60.96" y1="137.16" x2="-60.96" y2="144.78" width="0.1524" layer="91"/>
+<wire x1="-63.5" y1="139.7" x2="-60.96" y2="139.7" width="0.1524" layer="91"/>
+<wire x1="-60.96" y1="139.7" x2="-60.96" y2="144.78" width="0.1524" layer="91"/>
 <junction x="-60.96" y="144.78"/>
+<pinref part="H8" gate="G$1" pin="MOUNT"/>
+<wire x1="-60.96" y1="139.7" x2="-58.42" y2="139.7" width="0.1524" layer="91"/>
+<junction x="-60.96" y="139.7"/>
+<pinref part="H9" gate="G$1" pin="MOUNT"/>
+<wire x1="-60.96" y1="139.7" x2="-60.96" y2="132.08" width="0.1524" layer="91"/>
+<wire x1="-60.96" y1="132.08" x2="-58.42" y2="132.08" width="0.1524" layer="91"/>
+<pinref part="H7" gate="G$1" pin="MOUNT"/>
+<wire x1="-60.96" y1="132.08" x2="-63.5" y2="132.08" width="0.1524" layer="91"/>
+<junction x="-60.96" y="132.08"/>
+<pinref part="H10" gate="G$1" pin="MOUNT"/>
+<wire x1="-60.96" y1="149.86" x2="-60.96" y2="144.78" width="0.1524" layer="91"/>
 </segment>
 <segment>
